File: supply-use-one-wire-line-ac-hw/supply-use-one-wire-line-ac-hw.sch (KiCad schematic (older format))
At the start: 29 parts

Commit message: upload project
Parts:
- added C?: 100nF, symbol C
- added R?: 10k, Resistors_SMD:R_0805_HandSoldering, symbol R
- added Y?: Crystal, symbol Crystal
- C? (x2): value C -> 100nF
- C?: value C -> 1uF
Connections:
- net +5V: now also R?.1
- net GND: now also C?.2
- net Line: no longer Q?.2 (D), R?.2
- net supply: now also Q?.2 (D), R?.2
- net NRST: now reaches IC?.4 (NRST)
- net NRST: now also C?.1, R?.2
- net at IC?.5 (OSCIN/PA1): now also Y?.1
- net at IC?.6 (OSCOUT/PA2): now also Y?.2
Other:
- moved on the sheet: C?, U?
